File: hardware/AndyCabinets.kicad_pcb (KiCad board)
At the start: 2 copper layers, 33.9 x 104.5 mm, 50 parts

Commit message: Minor schematic cleanup
Connections:
- net /BRIGHT renamed /GPIO33_BRIGHT
- net /GPI34/BUT1 renamed /GPI34_BUT1_MODE
- net /GPI35 renamed /GPI35_SPEED
- net /GPI39 renamed /GPI39_COLOR
- net /GPIO32 renamed /GPIO32_PREVIEW
- R1 pad 2: +5V -> +3V3
- R6 pad 2: +5V -> +3V3
- RV1 pad 3: +5V -> +3V3
- RV2 pad 3: +5V -> +3V3
- S1 pad 1: +5V -> +3V3
- S2 pad 1: +5V -> +3V3
Routing:
- net +3V3: track 0.00 -> 122.1 mm, vias 0 -> 2
- net +5V: track 84.4 -> 71.1 mm
Other:
- board text added: "3.3v"
- board text added: "32 PREVIEW"
- board text added: "33 BRIGHT"
- board text added: "34 MODE"
- board text added: "35 SPEED"
- board text added: "39 COLOR"
- board text added: "5v"
- board text added: "BRIGHT"
- board text added: "COLOR"
- board text added: "EN"
- board text added: "GND"
- board text added: "GPIO 0"
- board text added: "HS2_CLK"
- board text added: "HS2_CMD"
- board text added: "HS2_DATA0"
- board text added: "I2C-SCL"
- board text added: "I2C-SDA"
- board text added: "MODE"
- board text added: "SPEED"
- board text added: "SPI_CS"
- board text added: "U0RXD"
- board text added: "U0TXD"
- board text added: "U1RXD"
- board text added: "U1TXD"
