File: hardware/AndyCabinets.sch (KiCad schematic (older format))
At the start: 50 parts

Commit message: Minor schematic cleanup
Connections:
- net BRIGHT renamed GPIO33_BRIGHT
- net GPI34/BUT1 renamed GPI34_BUT1_MODE
- net GPI35 renamed GPI35_SPEED
- net GPI39 renamed GPI39_COLOR
- net GPIO32 renamed GPIO32_PREVIEW
Other:
- moved on the sheet: C10, C11, C12, C13, C14, C15, C16, C17, C18, C3, C4, C5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

Commit message: Hardware: Rotary Encoder Play
Parts:
- removed C1, C2: 2.2uF, Capacitor_SMD:C_0805_2012Metric, symbol Device:C
- removed R1, R10, R2, R3, R4, R5, R6, R7, R8, R9: 1K, Resistor_SMD:R_0805_2012Metric, symbol Device:R
- removed S1, S2: RM106772BCB, YonaFootprints:RM106772BCB, symbol YonaSymbols:RM106772BCB
- added SW1: Mode_Encoder, symbol Device:Rotary_Encoder
- added SW?: Color_Encoder, symbol Device:Rotary_Encoder
Connections:
- net GPIO15/HS2_CMD is gone; now on net GPIO15_SPEED: EXT2.8
- net GPIO32_PREVIEW: no longer EXT2.6
- net GPI34_BUT1_MODE renamed GPIO34_MODE_A
- net GPIO34_MODE_A: now also SW?.A
- net GPI35_SPEED renamed GPIO15_SPEED
- net GPIO15_SPEED: no longer EXT2.3
- net GPI36/U1RXD renamed GPIO36_COLOR_B
- net GPIO36_COLOR_B: now also SW1.C
- net GPI39_COLOR renamed GPIO39_COLOR_A
- net GPIO39_COLOR_A: now also SW1.A
- net GPIO16/I2C-SCL renamed GPIO16_BRIGHT
- net GPIO16_BRIGHT: now also RV2.2
- net GPIO33_BRIGHT renamed GPIO33_MODE_B
- net GPIO33_MODE_B: now also SW?.C; no longer RV2.2
- new net GPIO32_MODE_C: EXT2.6, SW?.B
- new net GPIO35_COLOR_C: EXT2.3, SW1.B
- no-connect marks 13 -> 10
Other:
- moved on the sheet: RV2
