File: hardware/FaceplateBoard/FaceplateBoard.kicad_pcb (KiCad board)
At the start: 2 copper layers, 33.9 x 104.5 mm, 20 parts, among them SW1 Mode_Encoder, SW2 Color_Encoder

Commit message: After PCB v2
Other:
- board size 33.9 x 104.5 mm -> 33 x 104.5 mm
