File: hardware/IOBoard/AndyCabinets.sch (KiCad schematic (older format))
At the start: 50 parts, among them SW1 Mode_Encoder, SW2 Color_Encoder, U1 74HC14

Commit message: Rev 3 PCB
Parts:
- added J1: wESP Connector, YonaFootprints:PinSocket_2x10_P2.54mm_Vertical_SMD_Mirror, symbol Connector_Generic:Conn_02x10_Odd_Even
- added JP1: wESP Power Jumper, Jumper:SolderJumper-2_P1.3mm_Open_TrianglePad1.0x1.5mm, symbol Jumper:Jumper_2_Open
- SW1: value Mode_Encoder -> Color_Encoder; footprint Rotary_Encoder:RotaryEncoder_Alps_EC12E-Switch_Vertical_H20mm_CircularMountingHoles -> YonaFootprints:RotaryEncoder_Alps_EC12E-SMDSwitch_Vertical_H20mm_CircularMountingHoles
- SW2: value Color_Encoder -> Mode_Encoder
Connections:
- net +3V3: now also J1.2 (Pin_2)
- net +5V: now also JP1.2 (B)
- net GNDD: now also J1.1 (Pin_1), J1.19 (Pin_19), J1.9 (Pin_9)
- net GPIO13_SPEED renamed GPIO33
- net GPIO33: now also EXT2.5, J1.10 (Pin_10); no longer EXT2.10
- net GPIO14_PREVIEW renamed GPIO14
- net GPIO14: now also J1.14 (Pin_14)
- net GPIO15_BRIGHT renamed BRIGHT
- net BRIGHT: now also EXT2.4, J1.6 (Pin_6); no longer EXT2.8
- net GPIO32_COLOR_BTN renamed GPIO32
- net GPIO32: now also J1.7 (Pin_7)
- net GPIO33_COLOR_B renamed GPIO13
- net GPIO13: now also EXT2.10, J1.13 (Pin_13); no longer EXT2.5
- net GPIO34_COLOR_A renamed GPIO15
- net GPIO15: now also EXT2.8, J1.17 (Pin_17); no longer EXT2.4
- net GPIO35_MODE_BTN renamed COLOR_BTN
- net COLOR_BTN: now also J1.8 (Pin_8)
- net GPIO36_MODE_A renamed COLOR_A
- net COLOR_A: now also J1.4 (Pin_4)
- net GPIO39_MODE_B renamed COLOR_B
- net COLOR_B: now also J1.5 (Pin_5)
- new net GPIO12: J1.16 (Pin_16)
- new net GPIO18: J1.11 (Pin_11)
- new net GPIO2: J1.18 (Pin_18)
- new net GPIO23: J1.3 (Pin_3)
- new net GPIO4: J1.15 (Pin_15)
- new net GPIO5: J1.12 (Pin_12)
- new net wESP_V+: J1.20 (Pin_20), JP1.1 (A)
- no-connect marks 9 -> 15

Commit message: Hardware pre change to SMD2020
Parts:
- SW2: footprint Rotary_Encoder:RotaryEncoder_Alps_EC12E-Switch_Vertical_H20mm_CircularMountingHoles -> YonaFootprints:RotaryEncoder_Alps_EC12E-Switch_Vertical_H20mm_CircularMountingHoles_ReducedFootprint
Changed lines of the file:
@@
 F 0 "SW2" H 7750 6117 50  0000 C CNN
 F 1 "Mode_Encoder" H 7750 6026 50  0000 C CNN
-F 2 "Rotary_Encoder:RotaryEncoder_Alps_EC12E-Switch_Vertical_H20mm_CircularMountingHoles" H 7600 5910 50  0001 C CNN
+F 2 "YonaFootprints:RotaryEncoder_Alps_EC12E-Switch_Vertical_H20mm_CircularMountingHoles_ReducedFootprint" H 7600 5910 50  0001 C CNN
 F 3 "~" H 7750 6010 50  0001 C CNN
 	1    7750 5750
@@
 Wire Wire Line
 	2450 6400 3500 6400
-Connection ~ 3500 6500
-Connection ~ 3500 6400
-Connection ~ 3500 6100
-Connection ~ 3500 5900
-Connection ~ 900  6100
-Connection ~ 900  6300
-Connection ~ 900  6400
-Connection ~ 900  6500
-Connection ~ 900  6600
-Connection ~ 900  5800
 $EndSCHEMATC
